File: MeterReader_PCB/MCU.kicad_sch (KiCad schematic)
At the start: 4 parts, among them U2 E73-2G4M08S1C, Y1 32.768kHz

Commit message: move active components onto sensor PCB, finish layout of sensor PCB
Parts:
- C1, C2: footprint (none) -> Capacitor_SMD:C_0603_1608Metric
Connections:
- net Sensor_LED: now also U2.3 (P0.03/AIN1); no longer U2.6 (P1.13)
- net Button_1: now reaches U2.1 (P1.11)
- net UART_RX: now reaches U2.10 (P0.30/AIN6)
- net Button_2: now reaches U2.20 (P0.12)
- net VBUS: now reaches U2.27 (VBUS)
- net LED_2: now reaches U2.28 (P0.15)
- net Button_3: now reaches U2.35 (P0.24)
- net UART_TX: now reaches U2.9 (P0.31/AIN7)
- net LED renamed LED_0
